File: Iot_PCB/Projet_Iot/Projet_Iot.kicad_pcb (KiCad board)
At the start: 2 copper layers, 0 parts

Commit message: build(kicad) : start PCB
Parts:
- added D6: LED, LED_THT:LED_D5.0mm, F.Cu at (140.5, 89.9)
- added J10: 110990030, Grove:SEEED_110990030, F.Cu at (40.0, 131.8)
- added J11: 110990030, Grove:SEEED_110990030, F.Cu at (187.5, 38.7)
- added J12: 110990030, Grove:SEEED_110990030, F.Cu at (187.5, 45.4)
- added J13: 110990030, Grove:SEEED_110990030, F.Cu at (187.5, 52.0)
- added J14: 110990030, Grove:SEEED_110990030, F.Cu at (187.5, 58.7)
- added J15: 110990030, Grove:SEEED_110990030, F.Cu at (40.0, 138.4)
- added J16: 110990030, Grove:SEEED_110990030, F.Cu at (40.0, 145.1)
- added J17: 110990030, Grove:SEEED_110990030, F.Cu at (40.0, 151.7)
- added J18: 110990030, Grove:SEEED_110990030, F.Cu at (40.0, 158.3)
- added J21: Conn_01x15_Pin, Connector_PinHeader_2.54mm:PinHeader_1x15_P2.54mm_Vertical, F.Cu at (161.5, 38.9)
- added J22: Conn_01x15_Pin, Connector_PinHeader_2.54mm:PinHeader_1x15_P2.54mm_Vertical, F.Cu at (176.7, 38.1)
- added J23: 110990030, Grove:SEEED_110990030, F.Cu at (40.0, 165.0)
- added J24: 110990030, Grove:SEEED_110990030, F.Cu at (40.0, 171.7)
- added J36: 110990030, Grove:SEEED_110990030, F.Cu at (201.4, 80.9)
- added J37: 110990030, Grove:SEEED_110990030, F.Cu at (42.0, 63.3)
- added J38: 110990030, Grove:SEEED_110990030, F.Cu at (201.4, 87.5)
- added J39: 110990030, Grove:SEEED_110990030, F.Cu at (42.0, 70.0)
- added J40: 110990030, Grove:SEEED_110990030, F.Cu at (201.4, 94.2)
- added J41: 110990030, Grove:SEEED_110990030, F.Cu at (42.0, 76.6)
- added J42: 110990030, Grove:SEEED_110990030, F.Cu at (201.4, 100.8)
- added J43: 110990030, Grove:SEEED_110990030, F.Cu at (42.0, 83.2)
- added J6: 110990030, Grove:SEEED_110990030, F.Cu at (104.5, 26.0)
- added J7: 110990030, Grove:SEEED_110990030, F.Cu at (104.5, 32.6)
- added J8: 110990030, Grove:SEEED_110990030, F.Cu at (40.0, 118.5)
- added J9: 110990030, Grove:SEEED_110990030, F.Cu at (40.0, 125.1)
- added R14: 4700, Resistor_THT:R_Axial_DIN0207_L6.3mm_D2.5mm_P10.16mm_Horizontal, F.Cu at (194.9, 37.8)
- added R15: 10000, Resistor_THT:R_Axial_DIN0207_L6.3mm_D2.5mm_P10.16mm_Horizontal, F.Cu at (123.0, 89.9)
- added R16: R, Resistor_THT:R_Axial_DIN0207_L6.3mm_D2.5mm_P10.16mm_Horizontal, F.Cu at (140.8, 100.7)
- added U10: 74LS151, Package_DIP:DIP-16_W7.62mm, F.Cu at (49.4, 62.4)
- added U11: FDC6326L, FDC6326L:SOT95P280X110-6N, F.Cu at (155.0, 104.1)
- added U6: uPesy_ESP32_Wroom_Low_Power_DevKit, uPesyBoards:uPesy_ESP32_Wroom_Low_Power_DevKit, F.Cu at (107.5, 83.2)
- added U7: 74LS151, Package_DIP:DIP-16_W7.62mm, F.Cu at (208.8, 80.0)
Routing:
- net Net-(D6-A): track 0.00 -> 4.84 mm
- net Net-(U6-GPIO4): track 0.00 -> 4.10 mm
