File: Iot_PCB/Projet_Iot/Projet_Iot.kicad_sch (KiCad schematic)
At the start: 16 parts, among them J15 110990030, J16 110990030, J17 110990030, J18 110990030, J23 110990030, J24 110990030, J6 110990030, J7 Conn_01x04_Pin, U11 FDC6326L, U6 uPesy_ESP32_Wroom_Low_Power_D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

Commit message: final version of pcb
Connections:
- net ADC2: now reaches U6.3 (GPIO39)
- net ADC1: no longer names the net of U6.2 (GPIO36)
- net DHT22_IN: no longer names the net of U6.23 (GPIO18)
- no-connect marks 15 -> 16
Changed lines of the file:
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@@
 	)
 	(no_connect
-		(at 124.46 27.94)
+		(at 124.46 25.4)
 	)
 	(no_connect
@@
 	)
 	(no_connect
+		(at 161.29 38.1)
+	)
+	(no_connect
 		(at 124.46 43.18)
 	)
@@
 		)
 	)
-	(label "ADC1"
-		(at 124.46 25.4 180)
-		(effects
-			(font
-				(size 1.27 1.27)
-			)
-			(justify right bottom)
-		)
-	)
 	(label "Grove1-2"
 		(at 87.63 80.01 180)
@@
 		)
 	)
-	(label "ADC1"
+	(label "ADC2"
 		(at 97.79 57.15 0)
 		(effects
@@
 		)
 	)
-	(label "3v3"
+	(label "3v3_ESP"
 		(at 78.74 21.59 180)
 		(effects
@@
 		)
 	)
-	(label "DHT22_IN"
-		(at 161.29 38.1 0)
-		(effects
-			(font
-				(size 1.27 1.27)
-			)
-			(justify left bottom)
-		)
-	)
 	(label "interrupt_ia"
 		(at 158.75 35.56 0)
@@
 		(effects
 			(font
+				(size 1.27 1.27)
+			)
+			(justify right bottom)
+		)
+	)
+	(label "ADC2"
+		(at 124.46 27.94 180)
+		(effects
+			(font
