File: Iot_PCB/Projet_Iot/ventillateur_compmande.kicad_sch (KiCad schematic)
At the start: 3 parts, among them U7 EMC2301-x-ACZL

Commit message: final version of pcb
Parts:
- removed R8: 1200, symbol Device:R
- removed R9: 3300, symbol Device:R
- added U8: LDO40LPURY, Package_DFN_QFN:DFN-6-1EP_3x3mm_P0.95mm_EP1.7x2.6mm, symbol Regulator_Linear:LDO40LPURY
Connections:
- new net: U8.1 (GND), U8.7 (GND)
Other:
- moved on the sheet: U7
