File: Iot_PCB/PCB_ventillateur/controle_ventillateur/controle_ventillateur.kicad_pcb (KiCad board)
At the start: 2 copper layers, 37.6 x 34.5 mm, 5 parts, among them U7 EMC2301-x-ACZL

Commit message: pcb final version for both the gloabl projet and for the ventillator
Parts:
- added REF**: MountingHole_3.2mm_M3, MountingHole:MountingHole_3.2mm_M3, F.Cu at (189.7, 148.6)
- added REF**: CP_Radial_Tantal_D4.5mm_P2.50mm, Capacitor_THT:CP_Radial_Tantal_D4.5mm_P2.50mm, F.Cu at (192.7, 127.4)
- added REF**: R_Axial_DIN0207_L6.3mm_D2.5mm_P10.16mm_Horizontal, Resistor_THT:R_Axial_DIN0207_L6.3mm_D2.5mm_P10.16mm_Horizontal, F.Cu at (207.5, 129.2)
- added REF**: MountingHole_3.2mm_M3, MountingHole:MountingHole_3.2mm_M3, F.Cu at (189.6, 100.1)
- moved REF** 13.2 mm to (175.5, 136.4), turned to -90 degrees
Connections:
- DC/DC pad 3: /GND -> gnd_3.3
- Grove pad 1: /GND -> gnd_3.3
- U7 pad 4: /GND -> gnd_3.3
Routing:
- net /TACH: track 11.7 -> 62.7 mm
- net gnd_3.3: track 0.00 -> 47.8 mm
- net Net-(PS1-+VOUT): track 10.9 -> 30.1 mm
- net 12v: track 23.1 -> 37.3 mm
Other:
- board size 37.6 x 34.5 mm -> 45.7 x 62 mm

Commit message: correction pcb final
Connections:
- DC/DC pad 3: gnd_3.3 -> /GND
- Grove pad 1: gnd_3.3 -> /GND
- REF** pad 2: gnd_3.3 -> /GND
- U7 pad 4: gnd_3.3 -> /GND
Routing:
- net gnd_3.3: track 47.8 -> 0.00 mm
Changed lines of the file:
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@@
 	(net 8 "Net-(PS1-+VOUT)")
 	(net 9 "12v")
-	(net 10 "gnd_3.3")
 	(footprint "TerminalBlock_CUI:TerminalBlock_CUI_TB007-508-02_1x02_P5.08mm_Horizontal"
 		(layer "F.Cu")
@@
 			(layers "*.Cu" "*.Mask")
 			(remove_unused_layers no)
-			(net 10 "gnd_3.3")
+			(net 3 "/GND")
 		)
 		(embedded_fonts no)
@@
 			(layers "*.Cu" "*.Mask")
 			(remove_unused_layers no)
-			(net 10 "gnd_3.3")
+			(net 3 "/GND")
 			(solder_mask_margin 0.102)
 		)
@@
 			(layers "*.Cu" "*.Mask")
 			(remove_unused_layers no)
-			(net 10 "gnd_3.3")
+			(net 3 "/GND")
 			(solder_mask_margin 0.102)
 		)
@@
 			(layers "B.Cu" "B.Mask" "B.Paste")
 			(roundrect_rratio 0.25)
-			(net 10 "gnd_3.3")
+			(net 3 "/GND")
 			(pinfunction "GND")
 			(pintype "power_in")
@@
 		(net 9)
 	)
-	(segment
-		(start 189.952 127.174)
-		(end 192.659 129.881)
-		(width 0.4)
-		(layer "B.Cu")
-		(net 10)
-	)
-	(segment
-		(start 189.952 117.308)
-		(end 190.5805 116.6795)
-		(width 0.4)
-		(layer "B.Cu")
-		(net 10)
-	)
-	(segment
-		(start 189.952 122.4)
-		(end 189.952 117.308)
-		(width 0.4)
-		(layer "B.Cu")
-		(net 10)
-	)
-	(segment
-		(start 201.676 119.38)
-		(end 198.12 115.824)
-		(width 0.4)
-		(layer "B.Cu")
-		(net 10)
-	)
-	(segment
-		(start 192.659 129.881)
-		(end 193.138 130.36)
-		(width 0.4)
-		(layer "B.Cu")
-		(net 10)
-	)
-	(segment
-		(start 201.676 131.953)
-		(end 201.676 119.38)
-		(width 0.4)
-		(layer "B.Cu")
-		(net 10)
-	)
-	(segment
-		(start 192.659 129.881)
-		(end 192.659 131.064)
-		(width 0.4)
-		(layer "B.Cu")
-		(net 10)
-	)
-	(segment
-		(start 200.279 133.35)
-		(end 201.676 131.953)
-		(width 0.4)
-		(layer "B.Cu")
-		(net 10)
-	)
-	(segment
-		(start 190.5805 116.6795)
-		(end 190.5805 113.497)
-		(width 0.4)
-		(layer "B.Cu")
-		(net 10)
-	)
-	(segment
-		(start 189.952 122.4)
-		(end 189.952 127.174)
-		(width 0.4)
-		(layer "B.Cu")
-		(net 10)
-	)
-	(segment
-		(start 192.659 131.064)
-		(end 194.945 133.35)
-		(width 0.4)
-		(layer "B.Cu")
-		(net 10)
-	)
-	(segment
-		(start 194.945 133.35)
-		(end 200.279 133.35)
-		(width 0.4)
-		(layer "B.Cu")
-		(net 10)
-	)
 	(zone
